File: gpsdo/gpsdo.kicad_pcb (KiCad board)
At the start: 2 copper layers, 80 x 50 mm, 62 parts, among them IC1 ADP3335, IC2 STM32F405RxTx, IC3 NC7SZ04, IC4 CS2100-CP, IC5 MAX-M8Q, IC6 ADP3335, IC7 NCP380, P1 SWD_TC, P2 SMA, P3 SMA, P4 SMA, P5 SMA, P6 USB-B, Y1 26M, Y2 26M TCXO

Commit message: finished pcb
Parts:
- added TP5: TESTPAD, agg:TESTPAD, F.Cu at (156.2, 141.8)
- L1: footprint agg:0402-L -> agg:0402
- R6: footprint agg:0603 -> agg:0402
- moved C27 186.3 mm to (109.8, 139.4)
- moved R5 184.7 mm to (108.8, 144.4), turned to 90 degrees
- moved IC7 178.7 mm to (111.2, 143.4)
- moved D4 176.3 mm to (104.6, 133.8)
- moved R7 175.3 mm to (111.4, 127.2)
- moved C22 172.7 mm to (113.6, 143.2), turned to 270 degrees
- moved C25 162.4 mm to (116.0, 124.2), turned to 180 degrees
- moved C15 160.0 mm to (124.8, 122.8)
- moved TP1 153.9 mm to (142.0, 130.8)
- moved C26 151.7 mm to (108.4, 142.6), turned to 180 degrees
- moved C16 150.8 mm to (140.0, 128.0), turned to 90 degrees
- moved TP4 150.5 mm to (129.6, 143.2)
- moved C3 150.4 mm to (143.1, 121.9), turned to 270 degrees
- moved C9 149.1 mm to (144.0, 117.0), turned to 180 degrees
- moved C12 148.9 mm to (142.4, 139.2)
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Routing:
- net GND: track 0.00 -> 248.8 mm, vias 0 -> 235
- net 3v3: track 0.00 -> 154.8 mm, vias 0 -> 8
- net /GPS_PPS: track 0.00 -> 65.4 mm
- net /~FLAG: track 0.00 -> 42.4 mm, vias 0 -> 2
- net /~ANT_EN: track 0.00 -> 42.1 mm, vias 0 -> 2
- net /USART1_TX: track 0.00 -> 42.0 mm, vias 0 -> 2
- net /GPS_TIM1: track 0.00 -> 41.1 mm
- net /I2C1_SDA: track 0.00 -> 39.4 mm
- net /I2C1_SCL: track 0.00 -> 38.9 mm
- net /CLK_OUT_2: track 0.00 -> 37.8 mm
- net /USART1_RX: track 0.00 -> 37.3 mm
- net /STATUS: track 0.00 -> 34.4 mm, vias 0 -> 2
- net /GPS_RST: track 0.00 -> 28.2 mm, vias 0 -> 2
- net /CLK_OUT_1: track 0.00 -> 24.0 mm
- net /SWDIO: track 0.00 -> 23.8 mm, vias 0 -> 2
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- added copper zone on B.Cu, net GND
- added copper zone on F.Cu, net GND
Other:
- rule pad_to_mask_clearance: 0.2 -> 0
- rule via_min_drill: 0.3 -> 0.4
- rule via_min_size: 0.4 -> 0.8
- board text added: "CLK1"
- board text added: "CLK2"
- board text added: "GPSDO"
- board text added: "Matt Coates"
- board text added: "PPS"
- board text added: "PWR"
- board text added: "REF"
- board text added: "RX"
- board text added: "SCL"
- board text added: "SDA"
- board text added: "STAT"
- board text added: "TX"
- board text added: "v1"

Commit message: added external led
Parts:
- added J1: LED, agg:SIL-254P-02, F.Cu at (104.4, 126.2)
Routing:
- net Net-(D5-Pad2): track 3.07 -> 9.48 mm
- net GND: vias 235 -> 234
Changed lines of the file:
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@@
     (thickness 1.6)
     (drawings 29)
-    (tracks 713)
+    (tracks 714)
     (zones 0)
-    (modules 63)
+    (modules 64)
     (nets 85)
   )
@@
     )
   )
+  (module agg:SIL-254P-02 (layer F.Cu)
+    (at 104.4 126.2 90)
+    (fp_text reference J1 (at 0 -2.22 90) (layer F.Fab)
+      (effects (font (size 1 1) (thickness 0.15)))
+    )
+    (fp_text value LED (at 0 2.22 90) (layer F.Fab)
+      (effects (font (size 1 1) (thickness 0.15)))
+    )
+    (fp_line (start -2.54 -1.27) (end 2.54 -1.27) (layer F.Fab) (width 0.01))
+    (fp_line (start 2.54 -1.27) (end 2.54 1.27) (layer F.Fab) (width 0.01))
+    (fp_line (start 2.54 1.27) (end -2.54 1.27) (layer F.Fab) (width 0.01))
+    (fp_line (start -2.54 1.27) (end -2.54 -1.27) (layer F.Fab) (width 0.01))
+    (fp_line (start -2.54 -1.27) (end 2.54 -1.27) (layer F.SilkS) (width 0.15))
+    (fp_line (start 2.54 -1.27) (end 2.54 1.27) (layer F.SilkS) (width 0.15))
+    (fp_line (start 2.54 1.27) (end -2.54 1.27) (layer F.SilkS) (width 0.15))
+    (fp_line (start -2.54 1.27) (end -2.54 -1.27) (layer F.SilkS) (width 0.15))
+    (fp_line (start -2.8 -1.55) (end 2.8 -1.55) (layer F.CrtYd) (width 0.01))
+    (fp_line (start 2.8 -1.55) (end 2.8 1.55) (layer F.CrtYd) (width 0.01))
+    (fp_line (start 2.8 1.55) (end -2.8 1.55) (layer F.CrtYd) (width 0.01))
+    (fp_line (start -2.8 1.55) (end -2.8 -1.55) (layer F.CrtYd) (width 0.01))
+    (pad 1 thru_hole rect (at -1.27 0 90) (size 1.9 1.9) (drill 1) (layers *.Cu *.Mask F.SilkS)
+      (net 21 "Net-(D5-Pad2)"))
+    (pad 2 thru_hole circle (at 1.27 0 90) (size 1.9 1.9) (drill 1) (layers *.Cu *.Mask F.SilkS)
+      (net 2 GND))
+    (model ${KISYS3DMOD}/Pin_Headers.3dshapes/Pin_Header_Straight_1x02.wrl
+      (at (xyz 0 0 0))
+      (scale (xyz 1 1 1))
+      (rotate (xyz 0 0 0))
+    )
+  )
   (gr_text STAT (at 111.4 130.8) (layer F.SilkS)
     (effects (font (size 1 1) (thickness 0.15)))
@@
   (via (at 120 130) (size 0.8) (drill 0.4) (layers F.Cu B.Cu) (net 2))
   (via (at 110 135) (size 0.8) (drill 0.4) (layers F.Cu B.Cu) (net 2))
-  (via (at 105 125) (size 0.8) (drill 0.4) (layers F.Cu B.Cu) (net 2))
   (via (at 110 125) (size 0.8) (drill 0.4) (layers F.Cu B.Cu) (net 2))
   (via (at 110 120) (size 0.8) (drill 0.4) (layers F.Cu B.Cu) (net 2))
@@
   (via (at 132.2 131.2) (size 0.8) (drill 0.4) (layers F.Cu B.Cu) (net 2))
   (via (at 127.2 131.2) (size 0.8) (drill 0.4) (layers F.Cu B.Cu) (net 2))
-  (via (at 128.4 127.2) (size 0.8) (drill 0.4) (layers F.Cu B.Cu) (net 2) (status 1000000))
+  (via (at 128.4 127.2) (size 0.8) (drill 0.4) (layers F.Cu B.Cu) (net 2))
   (via (at 123.4 127.2) (size 0.8) (drill 0.4) (layers F.Cu B.Cu) (net 2))
   (segment (start 140.2 119.25) (end 138.35 119.25) (width 0.25) (layer F.Cu) (net 3))
@@
   (segment (start 110.7 127.8) (end 110.7 127.2) (width 0.25) (layer F.Cu) (net 21))
   (segment (start 110.9 128) (end 110.7 127.8) (width 0.25) (layer F.Cu) (net 21))
+  (segment (start 104.67 127.2) (end 104.4 127.47) (width 0.25) (layer F.Cu) (net 21))
+  (segment (start 110.7 127.2) (end 104.67 127.2) (width 0.25) (layer F.Cu) (net 21))
   (segment (start 116.3 127.2) (end 116.3 127.3) (width 0.25) (layer F.Cu) (net 22))
   (segment (start 116.3 127.9) (end 116.3 127.2) (width 0.25) (layer F.Cu) (net 22))
