File: gpsdo/gpsdo.sch (KiCad schematic (older format))
At the start: 67 parts, among them IC1 ADP3335, IC2 STM32F405RxTx, IC3 NC7SZ04, IC4 CS2100-CP, IC5 MAX-M8Q, IC6 ADP3335, IC7 NCP380, P1 SWD_TC, P2 SMA, P3 SMA, P4 SMA, P5 SMA, P6 USB-B, X1 Case, X2 Hole, X3 Hole, X4 Hole, X5 Hole, Y1 26M, Y2 26M TCXO

Commit message: finished pcb
Parts:
- removed X2, X3, X4, X5: Hole, agg:M3_HOLE, symbol agg-kicad:PART
- added TP5: TESTPAD, agg:TESTPAD, symbol agg-kicad:TESTPAD
- L1: footprint agg:0402-L -> agg:0402
- R6: footprint agg:0603 -> agg:0402; Farnell 1738878 -> 1652742
Connections:
- wire segments 279 -> 282
Changed lines of the file:
@@
 	6300 2900 6350 2900
 Wire Wire Line
-	6150 3900 6350 3900
+	6150 3900 6250 3900
 Wire Wire Line
 	6150 3600 6350 3600
@@
 $EndComp
 $Comp
-L agg-kicad:PART X2
-U 1 1 5B6C1661
-P 5500 7050
-F 0 "X2" H 5550 7150 50  0000 L CNN
-F 1 "Hole" H 5550 7050 50  0000 L CNN
-F 2 "agg:M3_HOLE" H 5500 7050 50  0001 C CNN
-F 3 "" H 5500 7050 50  0001 C CNN
-	1    5500 7050
-	1    0    0    -1
-$EndComp
-$Comp
-L agg-kicad:PART X3
-U 1 1 5B6C1817
-P 5500 7300
-F 0 "X3" H 5550 7400 50  0000 L CNN
-F 1 "Hole" H 5550 7300 50  0000 L CNN
-F 2 "agg:M3_HOLE" H 5500 7300 50  0001 C CNN
-F 3 "" H 5500 7300 50  0001 C CNN
-	1    5500 7300
-	1    0    0    -1
-$EndComp
-$Comp
-L agg-kicad:PART X4
-U 1 1 5B6C1887
-P 6050 7050
-F 0 "X4" H 6100 7150 50  0000 L CNN
-F 1 "Hole" H 6100 7050 50  0000 L CNN
-F 2 "agg:M3_HOLE" H 6050 7050 50  0001 C CNN
-F 3 "" H 6050 7050 50  0001 C CNN
-	1    6050 7050
-	1    0    0    -1
-$EndComp
-$Comp
-L agg-kicad:PART X5
-U 1 1 5B6C190D
-P 6050 7300
-F 0 "X5" H 6100 7400 50  0000 L CNN
-F 1 "Hole" H 6100 7300 50  0000 L CNN
-F 2 "agg:M3_HOLE" H 6050 7300 50  0001 C CNN
-F 3 "" H 6050 7300 50  0001 C CNN
-	1    6050 7300
-	1    0    0    -1
-$EndComp
-$Comp
 L agg-kicad:NCP380 IC7
 U 1 1 5B2067A4
@@
 F 0 "L1" H 10600 3750 50  0000 C CNN
 F 1 "27nH" H 10600 3650 50  0000 C CNN
-F 2 "agg:0402-L" H 10550 3700 50  0001 C CNN
+F 2 "agg:0402" H 10550 3700 50  0001 C CNN
 F 3 "" H 10550 3700 50  0001 C CNN
 F 4 "1343086" H 10550 3700 60  0001 C CNN "Farnell"
@@
 F 0 "R6" H 10400 3750 50  0000 C CNN
 F 1 "10" H 10400 3650 50  0000 C CNN
-F 2 "agg:0603" H 10350 3700 50  0001 C CNN
+F 2 "agg:0402" H 10350 3700 50  0001 C CNN
 F 3 "" H 10350 3700 50  0001 C CNN
-F 4 "1738878" H 10350 3700 60  0001 C CNN "Farnell"
+F 4 "1652742" H 10350 3700 60  0001 C CNN "Farnell"
 	1    10350 3700
 	-1   0    0    -1
@@
 	9250 5100 9350 5100
 Connection ~ 9350 5100
+$Comp
+L agg-kicad:TESTPAD TP5
+U 1 1 5B1FDC55
+P 6200 4000
+F 0 "TP5" H 6298 4000 50  0000 L CNN
+F 1 "TESTPAD" H 6200 3925 50  0001 L CNN
+F 2 "agg:TESTPAD" H 6200 3850 50  0001 L CNN
+F 3 "" H 6200 4000 50  0001 C CNN
+	1    6200 4000
+	-1   0    0    1
+$EndComp
+Wire Wire Line
+	6200 4000 6250 4000
+Wire Wire Line
+	6250 4000 6250 3900
+Connection ~ 6250 3900
+Wire Wire Line
+	6250 3900 6350 3900
 $EndSCHEMATC

Commit message: added external led
Parts:
- added J1: LED, agg:SIL-254P-02, symbol agg-kicad:CONN_01x02
Connections:
- wire segments 282 -> 286
Changed lines of the file:
@@
 L agg-kicad:LED D5
 U 1 1 5B201C70
-P 6150 6000
-F 0 "D5" V 6246 5942 50  0000 R CNN
-F 1 "LED" V 6155 5942 50  0000 R CNN
-F 2 "agg:0603-LED" H 6150 6000 50  0001 C CNN
-F 3 "" H 6150 6000 50  0001 C CNN
-F 4 "2290328" V 6150 6000 60  0001 C CNN "Farnell"
-	1    6150 6000
+P 6150 6050
+F 0 "D5" V 6246 5992 50  0000 R CNN
+F 1 "LED" V 6155 5992 50  0000 R CNN
+F 2 "agg:0603-LED" H 6150 6050 50  0001 C CNN
+F 3 "" H 6150 6050 50  0001 C CNN
+F 4 "2290328" V 6150 6050 60  0001 C CNN "Farnell"
+	1    6150 6050
 	0    -1   -1   0
 $EndComp
@@
 $EndComp
 Wire Wire Line
-	6150 6000 6150 6050
-Wire Wire Line
-	6150 5850 6150 5900
+	6150 6050 6150 6100
 Wire Wire Line
 	6150 5750 6150 5700
@@
 L agg-kicad:GND #PWR059
 U 1 1 5B2842A6
-P 6150 6050
-F 0 "#PWR059" H 6150 5800 50  0001 C CNN
-F 1 "GND" H 6150 5950 50  0000 C CNN
-F 2 "" H 6150 6050 50  0000 C CNN
-F 3 "" H 6150 6050 50  0000 C CNN
-	1    6150 6050
+P 6150 6100
+F 0 "#PWR059" H 6150 5850 50  0001 C CNN
+F 1 "GND" H 6150 6000 50  0000 C CNN
+F 2 "" H 6150 6100 50  0000 C CNN
+F 3 "" H 6150 6100 50  0000 C CNN
+	1    6150 6100
 	1    0    0    -1
 $EndComp
@@
 Wire Wire Line
 	6250 3900 6350 3900
+Wire Wire Line
+	6150 5850 6150 5900
+Wire Wire Line
+	6150 5900 5900 5900
+Connection ~ 6150 5900
+Wire Wire Line
+	6150 5900 6150 5950
+$Comp
+L agg-kicad:GND #PWR064
+U 1 1 5B23BCC3
+P 5950 6100
+F 0 "#PWR064" H 5950 5850 50  0001 C CNN
+F 1 "GND" H 5950 6000 50  0000 C CNN
+F 2 "" H 5950 6100 50  0000 C CNN
+F 3 "" H 5950 6100 50  0000 C CNN
+	1    5950 6100
+	1    0    0    -1
+$EndComp
+$Comp
+L agg-kicad:CONN_01x02 J1
+U 1 1 5B23C378
+P 5800 5900
+F 0 "J1" H 5800 6000 50  0000 C CNN
+F 1 "LED" H 5800 5700 50  0000 C CNN
+F 2 "agg:SIL-254P-02" H 5800 5900 50  0001 C CNN
+F 3 "" H 5800 5900 50  0001 C CNN
+F 4 "2112101" H 5800 5900 50  0001 C CNN "Farnell"
+	1    5800 5900
+	1    0    0    -1
+$EndComp
+Wire Wire Line
+	5950 6100 5950 6000
+Wire Wire Line
+	5950 6000 5900 6000
 $EndSCHEMATC
