File: gpsdo/pcb/gpsdo.sch (KiCad schematic (older format))
At the start: 65 parts, among them IC1 ADP3335, IC2 STM32F405RxTx, IC3 NC7SZ04, IC4 CS2100-CP, IC5 MAX-M8Q, IC6 ADP3335, IC7 NCP380, J1 LED, P1 SWD_TC, P2 SMA, P3 SMA, P4 SMA, P5 SMA, P6 USB-B, X1 Case, Y1 26M, Y2 26M TCXO

Commit message: added bom subs and gerbers zip
Parts:
- C16: Farnell 2496930 -> 2525102
- C2: Farnell 9402047 -> 2496771
- C22, C26: Farnell 2496814 -> 1758879
Changed lines of the file:
@@
 F 2 "agg:0603" H 2950 7300 50  0001 C CNN
 F 3 "" H 2950 7300 50  0000 C CNN
-F 4 "2496930" H 2950 7300 60  0001 C CNN "Farnell"
+F 4 "2525102" H 2950 7300 60  0001 C CNN "Farnell"
 	1    2950 7300
 	0    -1   -1   0
@@
 F 2 "agg:0402" H 1100 4100 50  0001 C CNN
 F 3 "" H 1100 4100 50  0000 C CNN
-F 4 "9402047" H 1100 4100 60  0001 C CNN "Farnell"
+F 4 "2496771" H 1100 4100 60  0001 C CNN "Farnell"
 	1    1100 4100
 	0    1    -1   0
@@
 F 2 "agg:0402" H 8450 3800 50  0001 C CNN
 F 3 "" H 8450 3800 50  0001 C CNN
-F 4 "2496814" H 8450 3800 60  0001 C CNN "Farnell"
+F 4 "1758879" H 8450 3800 60  0001 C CNN "Farnell"
 	1    8450 3800
 	0    -1   1    0
@@
 F 2 "agg:0402" H 10150 4100 50  0001 C CNN
 F 3 "" H 10150 4100 50  0001 C CNN
-F 4 "2496814" H 10150 4100 60  0001 C CNN "Farnell"
+F 4 "1758879" H 10150 4100 60  0001 C CNN "Farnell"
 	1    10150 4100
 	0    -1   1    0
